File: hardware/kicad/EveryDayCalendarSingleMonth.kicad_sch (KiCad schematic)
At the start: 57 parts, among them U3 74AHC1G125

Commit message: Move from RP2040 to ESP32, schematic mostly complete
Parts:
- removed D_S4: WS2812B, calendar:LED_WS2812C-2020-V1_2.0x2.0mm, symbol calendar:WS2812B
- removed SW_RESET1: Switch_SW_Push, calendar:SW_Push_1P1T_NO_6x6mm_H9.5mm, symbol tom-mechanical:SW_SPST
- added C? (x46): 1uF,25V,X5R, C_0402_1005Metric, symbol jlcpcb-basic-capacitor-0402:1uF,25V,X5R
- added C? (x9): 10uF,10V,X5R, C_0603_1608Metric, symbol jlcpcb-basic-capacitor-0603:10uF,10V,X5R
- added C? (x2): 1uF,25V,X5R, tom-passives:C_0402_1005Metric, symbol jlcpcb-basic-capacitor-0402:1uF,25V,X5R
- added D36, D37, D38, D39, D40, D41, D42: WS2812B, calendar:LED_WS2812C-2020-V1_2.0x2.0mm, symbol calendar:WS2812B
- added D?: LED, symbol Device:LED
- added J?: Conn_01x06, symbol Connector_Generic:Conn_01x06
- added J?: Conn_01x03, symbol Connector_Generic:Conn_01x03
- added Q? (x2): PN2222A, Package_TO_SOT_THT:TO-92_Inline, symbol Transistor_BJT:PN2222A
- added R? (x3): 10k, R_0402_1005Metric, symbol jlcpcb-basic-resistor-0402:10k
- added R?: 0, R_0402_1005Metric, symbol jlcpcb-basic-resistor-0402:0
- added R?: 1k, R_0402_1005Metric, symbol jlcpcb-basic-resistor-0402:1k
- added R?: 4.7k, R_0402_1005Metric, symbol jlcpcb-basic-resistor-0402:4.7k
- added SW_RESET, SW_RESET?, SW_WEEK6: Switch_SW_Push, calendar:SW_Push_1P1T_NO_6x6mm_H9.5mm, symbol tom-mechanical:SW_SPST
- added TP? (x12): TestPoint, TestPoint:TestPoint_Pad_2.5x2.5mm, symbol Connector:TestPoint
- added TP?: TestPoint, symbol Connector:TestPoint
- added U?: ESP32-WROOM-32E, RF_Module:ESP32-WROOM-32, symbol calendar:ESP32-WROOM-32E
- added VR?: LM1117MPX-3.3, tom-semiconductors:VREG_LM1117MPX-3.3, symbol tom-semiconductors:LM1117MPX-3.3
- SW_CAL_MODE1, SW_CAL_NEXT1, SW_CAL_PREV1, SW_DAY1, SW_DAY2, SW_DAY4, SW_DAY5, SW_DAY6, SW_DAY7, SW_WEEK1, SW_WEEK2, SW_WEEK3, SW_WEEK4, SW_WEEK5, SW_WIN1: LCSC C319395 -> C221880
- SW_DAY3: renamed from SW_dAY3; LCSC C319395 -> C221880
Connections:
- net VCC is gone; now on net +5V: U3.5 (VCC)
- net rp2040/GPIO1 is gone; now on net +5V: SW_DAY7.1 (A)
- net rp2040/GPIO10 is gone; now on net +5V: SW_WEEK3.1 (A)
- net rp2040/GPIO11 is gone; now on net +5V: SW_WEEK4.1 (A)
- net rp2040/GPIO12 is gone; now on net +5V: SW_WEEK5.1 (A)
- net rp2040/GPIO17 is gone; now on net +5V: SW_WIN1.1 (A)
- net rp2040/GPIO18 is gone; now on net +5V: SW_CAL_MODE1.1 (A)
- net rp2040/GPIO19 is gone; now on net +5V: SW_CAL_NEXT1.1 (A)
- net rp2040/GPIO2 is gone; now on net +5V: SW_DAY6.1 (A)
- net rp2040/GPIO20 is gone; now on net +5V: SW_CAL_PREV1.1 (A)
- net rp2040/GPIO3 is gone; now on net +5V: SW_DAY5.1 (A)
- net rp2040/GPIO4 is gone; now on net +5V: SW_DAY4.1 (A)
- net rp2040/GPIO5 is gone; now on net +5V: SW_DAY3.1 (A)
- net rp2040/GPIO6 is gone; now on net +5V: SW_DAY2.1 (A)
- net rp2040/GPIO7 is gone; now on net +5V: SW_DAY1.1 (A)
- net rp2040/GPIO8 is gone; now on net +5V: SW_WEEK1.1 (A)
- net rp2040/GPIO9 is gone; now on net +5V: SW_WEEK2.1 (A)
- net +5V: now also D1.2 (VSS), D10.2 (VSS), D11.2 (VSS), D12.2 (VSS), D13.2 (VSS), D14.2 (VSS), D15.2 (VSS), D16.2 (VSS), D17.2 (VSS), D18.2 (VSS), D19.2 (VSS), D2.2 (VSS), D20.2 (VSS), D21.2 (VSS), D22.2 (VSS), D23.2 (VSS), D24.2 (VSS), D25.2 (VSS), D26.2 (VSS), D27.2 (VSS), D28.2 (VSS), D29.2 (VSS), D3.2 (VSS), D30.2 (VSS), D31.2 (VSS), D32.2 (VSS), D33.2 (VSS), D34.2 (VSS), D35.2 (VSS), D4.2 (VSS), D5.2 (VSS), D6.2 (VSS), D7.2 (VSS), D8.2 (VSS), D9.2 (VSS), D_S1.2 (VSS), D_S2.2 (VSS), D_S3.2 (VSS), U3.1, U3.3 (GND), C?.1, C?.1, C?.1, C?.1, C?.1, C?.1, C?.1, C?.1, C?.1, C?.1, C?.1, C?.1, C?.1, C?.1, C?.1, C?.1, C?.1, C?.1, C?.1, C?.1, C?.1, C?.1, C?.1, C?.1, C?.1, C?.1, C?.1, C?.1, C?.1, C?.1, C?.1, C?.1, C?.1, C?.1, C?.1, C?.1, C?.1, C?.1, C?.1, C?.1, C?.1, C?.1, C?.1, C?.1, C?.1, C?.1, C?.1, C?.1, C?.1, C?.1, C?.1, C?.1, C?.1, C?.2, C?.2, C?.2, C?.2, C?.2, C?.2, C?.2, C?.2, C?.2, C?.2, C?.2, C?.2, C?.2, C?.2, C?.2, C?.2, C?.2, C?.2, C?.2, C?.2, C?.2, C?.2, C?.2, C?.2, C?.2, C?.2, C?.2, C?.2, C?.2, C?.2, C?.2, C?.2, C?.2, C?.2, C?.2, C?.2, C?.2, C?.2, C?.2, C?.2, C?.2, C?.2, C?.2, C?.2, C?.2, C?.2, C?.2, C?.2, C?.2, C?.2, C?.2, C?.2, C?.2, C?.2, C?.2, C?.2, C?.2, D36.2 (VSS), D36.4 (VDD), D37.2 (VSS), D37.4 (VDD), D38.2 (VSS), D38.4 (VDD), D39.2 (VSS), D39.4 (VDD), D40.2 (VSS), D40.4 (VDD), D41.2 (VSS), D41.4 (VDD), D42.2 (VSS), D42.4 (VDD), D?.1 (K), J?.1 (Pin_1), J?.3 (Pin_3), J?.3 (Pin_3), SW_RESET.2 (B), SW_RESET?.2 (B), SW_WEEK6.1 (A), TP?.1, TP?.1, TP?.1, TP?.1, TP?.1, TP?.1, TP?.1, TP?.1, U?.1 (GND), U?.15 (GND), U?.38 (GND), U?.39 (GND), VR?.1 (GND), VR?.3 (VIN)
- net at D1.3 (DIN): now also D_S3.1 (DOUT)
- net at D35.1 (DOUT): now also D36.3 (DIN)
- removed net GND: D1.2 (VSS), D10.2 (VSS), D11.2 (VSS), D12.2 (VSS), D13.2 (VSS), D14.2 (VSS), D15.2 (VSS), D16.2 (VSS), D17.2 (VSS), D18.2 (VSS), D19.2 (VSS), D2.2 (VSS), D20.2 (VSS), D21.2 (VSS), D22.2 (VSS), D23.2 (VSS), D24.2 (VSS), D25.2 (VSS), D26.2 (VSS), D27.2 (VSS), D28.2 (VSS), D29.2 (VSS), D3.2 (VSS), D30.2 (VSS), D31.2 (VSS), D32.2 (VSS), D33.2 (VSS), D34.2 (VSS), D35.2 (VSS), D4.2 (VSS), D5.2 (VSS), D6.2 (VSS), D7.2 (VSS), D8.2 (VSS), D9.2 (VSS), D_S1.2 (VSS), D_S2.2 (VSS), D_S3.2 (VSS), SW_CAL_MODE1.2 (B), SW_CAL_NEXT1.2 (B), SW_CAL_PREV1.2 (B), SW_DAY1.2 (B), SW_DAY2.2 (B), SW_DAY3.2 (B), SW_DAY4.2 (B), SW_DAY5.2 (B), SW_DAY6.2 (B), SW_DAY7.2 (B), SW_WEEK1.2 (B), SW_WEEK2.2 (B), SW_WEEK3.2 (B), SW_WEEK4.2 (B), SW_WEEK5.2 (B), SW_WIN1.2 (B), U3.1, U3.3 (GND)
- net rp2040/GPIO15 renamed LED_LINK
- net LED_LINK: now also R?.2, TP?.1, TP?.1, TP?.1, TP?.1
- new net: Q?.2 (B), R?.2 (x2)
- new net: D37.1 (DOUT), D38.3 (DIN)
- new net: D36.1 (DOUT), D37.3 (DIN)
- new net: D?.2 (A), R?.1
- new net: D41.1 (DOUT), D42.3 (DIN)
- new net: D40.1 (DOUT), D41.3 (DIN)
- new net: D38.1 (DOUT), D39.3 (DIN)
- new net: D39.1 (DOUT), D40.3 (DIN)
- new net: J?.2 (Pin_2), R?.1
- new net +3.3V: C?.1, C?.1, C?.1, J?.1 (Pin_1), R?.2, U?.2 (VDD), VR?.2 (VOUT_2), VR?.4 (VOUT_4)
- new net BUTTON_CAL_NEXT: SW_CAL_NEXT1.2 (B), U?.8 (IO32)
- new net BUTTON_CAL_PREV: SW_CAL_PREV1.2 (B), U?.12 (IO27)
- new net BUTTON_MODE: SW_CAL_MODE1.2 (B), U?.6 (IO34)
- new net BUTTON_WIN: SW_WIN1.2 (B), U?.7 (IO35)
- new net DAY1: SW_DAY1.2 (B), U?.29 (IO5)
- new net DAY2: SW_DAY2.2 (B), SW_DAY3.2 (B), U?.14 (IO12)
- new net DAY3: SW_DAY4.2 (B), U?.13 (IO14)
- new net DAY4: SW_DAY5.2 (B), U?.23 (IO15)
- new net DAY5: SW_DAY6.2 (B), U?.27 (IO16)
- new net DAY6: SW_DAY7.2 (B), U?.28 (IO17)
- new net DAY7: U?.30 (IO18)
- new net DTR: Q?.1 (E), R?.1
- new net GPIO0: Q?.3 (C), SW_RESET?.1 (A), U?.25 (IO0)
- new net PIN_LED: R?.1
- new net PIN_LED_CAL: U?.9 (IO33)
- new net PIN_LED_STATUS: R?.2, U?.16 (IO13)
- new net PIN_ONE_WIRE: R?.2, U?.24 (IO2)
- new net PIN_TEST_POINT: TP?.1, U?.26 (IO4)
- new net RESET: C?.1, Q?.3 (C), R?.1, SW_RESET.1 (A), U?.3 (EN)
- new net RTS: J?.6 (Pin_6), Q?.1 (E), R?.1
- new net RXD: J?.4 (Pin_4)
- new net TXD: J?.5 (Pin_5)
- new net WEEK1: SW_WEEK1.2 (B), U?.31 (IO19)
- new net WEEK2: SW_WEEK2.2 (B), U?.33 (IO21)
- new net WEEK3: SW_WEEK3.2 (B), U?.36 (IO22)
- new net WEEK4: SW_WEEK4.2 (B), U?.37 (IO23)
- new net WEEK5: SW_WEEK5.2 (B), U?.10 (IO25)
- new net WEEK6: SW_WEEK6.2 (B), U?.11 (IO26)
- no-connect marks 0 -> 3
Other:
- removed sheet rp2040
- moved on the sheet: D1, D10, D11, D12, D13, D14, D15, D16, D17, D18, D19, D2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

Commit message: Schematic complete, pcb outline in place
Parts:
- removed VR?: LM1117MPX-3.3, tom-semiconductors:VREG_LM1117MPX-3.3, symbol tom-semiconductors:LM1117MPX-3.3
- added J2: Conn_01x02, Connector_Phoenix_MC:PhoenixContact_MCV_1,5_2-G-3.81_1x02_P3.81mm_Vertical, symbol Connector_Generic:Conn_01x02
- added TP15, TP16, TP17, TP18: TestPoint, MountingHole:MountingHole_3.2mm_M3, symbol Connector:TestPoint
- added TP2: TestPoint, TestPoint:TestPoint_Pad_2.5x2.5mm, symbol Connector:TestPoint
- added U3: LT1117-3.3, Package_TO_SOT_SMD:TO-263-3_TabPin2, symbol Regulator_Linear:LT1117-3.3
- C1, C10, C3, C4, C5, C6, C7, C8, C9: renamed from C?; footprint C_0603_1608Metric -> tom-passives:C_0603_1608Metric
- C11, C12, C13, C14, C15, C16, C17, C19, C20, C21, C22, C23, C24, C25, C26, C27, C28, C29, C30, C31, C32, C33, C34, C35, C36, C37, C38, C39, C40, C41, C42, C43, C44, C45, C46, C47, C48, C49, C50, C51, C52, C53, C54, C55, C56, C57: renamed from C?; footprint C_0402_1005Metric -> tom-passives:C_0402_1005Metric
- D19: renamed from D?; footprint (none) -> tom-opto:LED_0603_1608Metric; LCSC (none) -> C2286
- J1: renamed from J?; footprint (none) -> Connector_PinHeader_2.54mm:PinHeader_1x03_P2.54mm_Vertical
- J3: renamed from J?; footprint (none) -> Connector_PinHeader_2.54mm:PinHeader_1x06_P2.54mm_Vertical
- Q1, Q2: renamed from Q?; footprint Package_TO_SOT_THT:TO-92_Inline -> Package_TO_SOT_SMD:SOT-23; LCSC (none) -> C242260
- R1, R2, R3, R4, R5, R6: renamed from R?; footprint R_0402_1005Metric -> tom-passives:R_0402_1005Metric
- TP1: renamed from TP?; footprint (none) -> TestPoint:TestPoint_Pad_D2.0mm
- gave numbers to parts that had none: 16
- renumbered D23 to D10, D30 to D11, D37 to D12, D3 to D13, D10 to D14, D17 to D15, D24 to D16, D31 to D17, D38 to D18, D8 to D2, D4 to D20, D11 to D21, D18 to D22, D25 to D23, D32 to D24, D39 to D25, D5 to D26, D12 to D27, D19 to D28, D26 to D29, D15 to D3, D33 to D30, D40 to D31, D6 to D32, D13 to D33, D20 to D34, D27 to D35, D34 to D36, D41 to D37, D7 to D38, D14 to D39, D22 to D4, D21 to D40, D28 to D41, D35 to D42, D42 to D43, D29 to D5, D36 to D6, D2 to D7, D9 to D8, D16 to D9, SW_DAY7 to SW_DAY1, SW_DAY6 to SW_DAY2, SW_DAY5 to SW_DAY3, SW_DAY3 to SW_DAY5, SW_DAY2 to SW_DAY6, SW_DAY1 to SW_DAY7, SW_RESET to SW_RESET2, U3 to U2
Connections:
- net PIN_LED is gone; now on net PIN_LED_CAL: R1.1
- net +3.3V: now also U3.2 (VO)
- net +5V: now also J2.1 (Pin_1), U3.3 (VI); no longer C1.2, C10.2, C11.2, C12.2, C13.2, C14.2, C15.2, C16.2, C17.2, C18.2, C19.2, C2.2, C20.2, C21.2, C22.2, C23.2, C24.2, C25.2, C26.2, C27.2, C28.2, C29.2, C3.1, C30.2, C31.2, C32.2, C33.2, C34.2, C35.2, C36.2, C37.2, C38.2, C39.2, C4.1, C40.2, C41.2, C42.2, C43.2, C44.2, C45.2, C46.2, C47.2, C48.2, C49.2, C5.1, C50.2, C51.2, C52.2, C53.2, C54.2, C55.2, C56.2, C57.2, C6.1, C7.1, C8.1, C9.1, D1.2 (VSS), D10.2 (VSS), D11.2 (VSS), D12.2 (VSS), D13.2 (VSS), D14.2 (VSS), D15.2 (VSS), D16.2 (VSS), D17.2 (VSS), D18.2 (VSS), D19.1 (K), D2.2 (VSS), D20.2 (VSS), D21.2 (VSS), D22.2 (VSS), D23.2 (VSS), D24.2 (VSS), D25.2 (VSS), D26.2 (VSS), D27.2 (VSS), D28.2 (VSS), D29.2 (VSS), D3.2 (VSS), D30.2 (VSS), D31.2 (VSS), D32.2 (VSS), D33.2 (VSS), D34.2 (VSS), D35.2 (VSS), D36.2 (VSS), D37.2 (VSS), D38.2 (VSS), D39.2 (VSS), D4.2 (VSS), D40.2 (VSS), D41.2 (VSS), D42.2 (VSS), D43.2 (VSS), D5.2 (VSS), D6.2 (VSS), D7.2 (VSS), D8.2 (VSS), D9.2 (VSS), D_S1.2 (VSS), D_S2.2 (VSS), D_S3.2 (VSS), J1.3 (Pin_3), J3.1 (Pin_1), SW_CAL_MODE1.1 (A), SW_CAL_NEXT1.1 (A), SW_CAL_PREV1.1 (A), SW_DAY1.1 (A), SW_DAY2.1 (A), SW_DAY3.1 (A), SW_DAY4.1 (A), SW_DAY5.1 (A), SW_DAY6.1 (A), SW_DAY7.1 (A), SW_RESET1.2 (B), SW_RESET2.2 (B), SW_WEEK1.1 (A), SW_WEEK2.1 (A), SW_WEEK3.1 (A), SW_WEEK4.1 (A), SW_WEEK5.1 (A), SW_WEEK6.1 (A), SW_WIN1.1 (A), TP10.1, TP5.1, TP6.1, TP9.1, U1.1 (GND), U1.15 (GND), U1.38 (GND), U1.39 (GND), U2.1, U2.3 (GND), U2.5 (VCC)
- net DAY1: now also SW_DAY1.2 (B); no longer SW_DAY7.2 (B)
- net DAY2: now also SW_DAY2.2 (B); no longer SW_DAY5.2 (B), SW_DAY6.2 (B)
- net DAY3: now also SW_DAY3.2 (B); no longer SW_DAY4.2 (B)
- net DAY4: now also SW_DAY4.2 (B); no longer SW_DAY3.2 (B)
- net DAY5: now also SW_DAY5.2 (B); no longer SW_DAY2.2 (B)
- net DAY6: now also SW_DAY6.2 (B); no longer SW_DAY1.2 (B)
- net DAY7: now also SW_DAY7.2 (B)
- net RXD: now also U1.34 (RXD0/IO3)
- net TXD: now also U1.35 (TXD0/IO1)
- net at D38.3 (DIN): now also D32.1 (DOUT)
- net at D43.1 (DOUT): now also TP2.1
- new net GND: C1.2, C10.2, C11.2, C12.2, C13.2, C14.2, C15.2, C16.2, C17.2, C18.2, C19.2, C2.2, C20.2, C21.2, C22.2, C23.2, C24.2, C25.2, C26.2, C27.2, C28.2, C29.2, C3.1, C30.2, C31.2, C32.2, C33.2, C34.2, C35.2, C36.2, C37.2, C38.2, C39.2, C4.1, C40.2, C41.2, C42.2, C43.2, C44.2, C45.2, C46.2, C47.2, C48.2, C49.2, C5.1, C50.2, C51.2, C52.2, C53.2, C54.2, C55.2, C56.2, C57.2, C6.1, C7.1, C8.1, C9.1, D1.2 (VSS), D10.2 (VSS), D11.2 (VSS), D12.2 (VSS), D13.2 (VSS), D14.2 (VSS), D15.2 (VSS), D16.2 (VSS), D17.2 (VSS), D18.2 (VSS), D19.1 (K), D2.2 (VSS), D20.2 (VSS), D21.2 (VSS), D22.2 (VSS), D23.2 (VSS), D24.2 (VSS), D25.2 (VSS), D26.2 (VSS), D27.2 (VSS), D28.2 (VSS), D29.2 (VSS), D3.2 (VSS), D30.2 (VSS), D31.2 (VSS), D32.2 (VSS), D33.2 (VSS), D34.2 (VSS), D35.2 (VSS), D36.2 (VSS), D37.2 (VSS), D38.2 (VSS), D39.2 (VSS), D4.2 (VSS), D40.2 (VSS), D41.2 (VSS), D42.2 (VSS), D43.2 (VSS), D5.2 (VSS), D6.2 (VSS), D7.2 (VSS), D8.2 (VSS), D9.2 (VSS), D_S1.2 (VSS), D_S2.2 (VSS), D_S3.2 (VSS), J1.3 (Pin_3), J2.2 (Pin_2), J3.1 (Pin_1), SW_CAL_MODE1.1 (A), SW_CAL_NEXT1.1 (A), SW_CAL_PREV1.1 (A), SW_DAY1.1 (A), SW_DAY2.1 (A), SW_DAY3.1 (A), SW_DAY4.1 (A), SW_DAY5.1 (A), SW_DAY6.1 (A), SW_DAY7.1 (A), SW_RESET1.2 (B), SW_RESET2.2 (B), SW_WEEK1.1 (A), SW_WEEK2.1 (A), SW_WEEK3.1 (A), SW_WEEK4.1 (A), SW_WEEK5.1 (A), SW_WEEK6.1 (A), SW_WIN1.1 (A), TP10.1, TP15.1, TP16.1, TP17.1, TP18.1, TP5.1, TP6.1, TP9.1, U1.1 (GND), U1.15 (GND), U1.38 (GND), U1.39 (GND), U2.1, U2.3 (GND), U3.1 (GND)
- new net VCC: U2.5 (VCC)
Other:
- note added: "TODO: Fix power to U2"
