File: hardware/kicad/EveryDayCalendarSingleMonth.kicad_pcb (KiCad board)
At the start: 2 copper layers, 100 x 100 mm, 147 parts, among them J2_POWER_IN1 Conn_01x02, J3_PROGRAMING_PIN1 Conn_01x06, Q1 PN2222A, Q2 PN2222A, U1 74AHC1G125

Commit message: Keep optimizing the tracks
Parts:
- moved C41 3.91 mm to (133.0, 97.5), turned to 0 degrees
- moved C39 3.90 mm to (133.5, 78.0), turned to 0 degrees
- moved C40 3.72 mm to (133.2, 87.5), turned to 0 degrees
- moved C2 3.51 mm to (133.0, 130.8)
- moved C38 3.19 mm to (134.0, 67.5), turned to 0 degrees
- moved C19 1.96 mm to (106.5, 56.2), turned to 0 degrees
- moved C31 1.96 mm to (128.5, 56.2), turned to 0 degrees
- moved C25 1.95 mm to (117.5, 56.2), turned to 0 degrees
- moved C13 1.60 mm to (95.0, 56.2), turned to 0 degrees
- moved C4 1.46 mm to (83.8, 56.2), turned to 0 degrees
- moved C37 1.27 mm to (135.8, 56.2), turned to 0 degrees
- moved ROW1 1.25 mm to (72.8, 56.0), turned to 180 degrees
Routing:
- net +5V: track 827.5 -> 801.1 mm
- net Net-(DAY35-Pad1): track 85.9 -> 78.6 mm
- net Net-(DAY28-Pad1): track 86.3 -> 79.3 mm
- net Net-(DAY21-Pad1): track 85.1 -> 78.6 mm
- net Net-(DAY14-Pad1): track 85.7 -> 79.5 mm
- net GND: track 188.9 -> 191.3 mm
- net Net-(DAY1-Pad1): track 10.8 -> 9.63 mm
- net /DAY1: track 135.3 -> 136.1 mm
- net Net-(DAY7-Pad1): track 85.4 -> 84.6 mm
- net Net-(DAY5-Pad1): track 10.4 -> 9.63 mm
- net Net-(DAY4-Pad1): track 10.4 -> 9.63 mm
- net Net-(DAY3-Pad1): track 10.4 -> 9.60 mm
- net Net-(DAY6-Pad1): track 10.4 -> 9.64 mm
- net Net-(DAY2-Pad1): track 10.4 -> 9.65 mm
Other:
- board text added: "Motivation is what gets you started Habit is what keeps you going -- Jim Ryun"

Commit message: Added gerber files
Routing:
- net GND: track 191.3 -> 212.5 mm
- net +3.3V: track 83.1 -> 76.9 mm, vias 4 -> 9
- added copper zone on B.Cu, net +3.3V
- added copper zone on F.Cu, net +3.3V
